File: Episode06/hexdisplay16/hexdisplay16.sch (KiCad schematic (older format))
At the start: 28 parts, among them J1 Conn_01x06_Male, J2 Conn_01x05_Male, J3 Conn_01x05_Male, J4 Conn_01x05_Male, J5 Conn_01x05_Male, J6 Conn_01x05_Male, J7 Conn_01x05_Male, J8 Conn_01x05_Male, J9 Conn_01x05_Male, Q1 MMBT3906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

Commit message: only use local symbol libraries
Parts:
- removed J1: Conn_01x06_Male, symbol Connector:Conn_01x06_Male
- removed J2, J3, J4, J5, J6, J7, J8, J9: Conn_01x05_Male, symbol Connector:Conn_01x05_Male
- removed J?: Conn_01x02_Male, symbol Connector:Conn_01x02_Male
- removed J?: Conn_01x16_Male, symbol Connector:Conn_01x16_Male
- added J1, J2, J3, J4, J5, J6, J7, J8: Conn_01x05, symbol Connector_Generic:Conn_01x05
- added J10: Conn_01x16, symbol Connector_Generic:Conn_01x16
- added J9: Conn_01x02, symbol Connector_Generic:Conn_01x02
- added J?: Conn_01x06, symbol Connector_Generic:Conn_01x06
- R1, R2, R3, R4, R5, R6, R7: value 680 -> 330
