File: Episode06/hexdisplay8/hexdisplay8.sch (KiCad schematic (older format))
At the start: 18 parts, among them J1 Conn_02x05_Counter_Clockwise, J2 Conn_02x05_Counter_Clockwise, J3 Conn_01x02, J4 Conn_01x08, J5 Conn_01x06, Q1 MMBT3906, Q2 MMBT3906, U1 ATTINY2313A-SU

Commit message: minor schematic updates, regenerated PDFs
Other:
- note added: "Resistance of R1-R7 should\nbe adjusted based on brightness\nof LED displays. (330 Ohms is\nlikely too high for standard\nLEDs.)"
Changed lines of the file:
@@
 Wire Wire Line
 	2300 1950 2300 2050
+Text Notes 3600 4350 0    50   ~ 0
+Resistance of R1-R7 should\nbe adjusted based on brightness\nof LED displays.  (330 Ohms is\nlikely too high for standard\nLEDs.)
 $EndSCHEMATC
