File: Episode08/hexdisplay8/hexdisplay8.kicad_pcb (KiCad board)
At the start: 2 copper layers, 51.9 x 23.8 mm, 20 parts, among them J11 Conn_01x05, J12 Conn_01x05, J21 Conn_01x05, J22 Conn_01x05, J3 Conn_01x02, J4 Conn_01x08, J5 Conn_01x06, Q1 MMBT3906, Q2 MMBT3906, U1 ATTINY2313A-SU

Commit message: regenerate gerbers
JLCPCB is giving me issues. Probably will just order and
hope for the best, the boards seem file when viewed in KiCad's
gerber viewer.
Routing:
- added copper zone on B.Cu, net GND
- added copper zone on F.Cu, net GND
- removed copper zone on B.Cu, net (none)
- removed copper zone on F.Cu, net (none)
