File: Episode09/hexdisplay16/hexdisplay16.kicad_pcb (KiCad board)
At the start: 2 copper layers, 63.7 x 24.6 mm, 28 parts, among them J11 Conn_01x05, J12 Conn_01x05, J21 Conn_01x05, J22 Conn_01x05, J31 Conn_01x05, J32 Conn_01x05, J41 Conn_01x05, J42 Conn_01x05, J5 Conn_01x02, J6 Conn_01x16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

Commit message: updated URL on silkscreen
The hex display episode will be Random Stuff #9.
Unfortunately, the actual PCBs say Episode 08. Oh well.
Other:
- board text added: "https://github.com/daveho/RandomStuff/ tree/master/Episode09/hexdisplay16"
- board text removed: "https://github.com/daveho/RandomStuff/ tree/master/Episode08/hexdisplay16"
