File: Episode0a/SunBladeNVRAM/SunBladeNVRAM.kicad_sch (KiCad schematic)
At the start: 15 parts, among them J1 Conn_01x14_Pin, J105 Conn_01x01_Pin, J106 Conn_01x01_Pin, J107 Conn_01x01_Pin, J108 Conn_01x01_Pin, J2 Conn_01x14_Pin, J3 Conn_01x02_Pin, J4 Conn_01x02_Pin, J5 Conn_01x01_Pin, J6 Conn_01x01_Pin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

Commit message: remove xtal from bottom PCB
There's no point in wiring the xtal to the bottom PCB
since it can be soldered directly to the snap connectors
on the M48T59Y-70MH1.

Also, increase the size of the "notch" arc on the bottom
PCB, and add it to the top PCB.
Parts:
- removed J3: Conn_01x02_Pin, Connector_PinHeader_2.54mm:PinHeader_1x02_P2.54mm_Vertical, symbol Connector:Conn_01x02_Pin
- removed Y1: 32.768 kHz, Crystal:Crystal_C38-LF_D3.0mm_L8.0mm_Horizontal, symbol Device:Crystal
Changed lines of the file:
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@@
-	(wire
-		(pts
-			(xy 54.61 130.81) (xy 54.61 139.7)
-		)
-		(stroke
-			(width 0)
-			(type default)
-		)
-	)
 	(wire
 		(pts
@@
 	(wire
 		(pts
-			(xy 46.99 130.81) (xy 46.99 139.7)
-		)
-		(stroke
-			(width 0)
-			(type default)
-		)
-	)
-	(wire
-		(pts
 			(xy 49.53 81.28) (xy 64.77 81.28)
 		)
@@
 	(wire
 		(pts
-			(xy 54.61 139.7) (xy 52.07 139.7)
-		)
-		(stroke
-			(width 0)
-			(type default)
-		)
-	)
-	(wire
-		(pts
 			(xy 102.87 78.74) (xy 118.11 78.74)
 		)
@@
 	(wire
 		(pts
-			(xy 46.99 139.7) (xy 49.53 139.7)
-		)
-		(stroke
-			(width 0)
-			(type default)
-		)
-	)
-	(wire
-		(pts
 			(xy 49.53 88.9) (xy 64.77 88.9)
 		)
@@
 	)
 	(rectangle
-		(start 43.18 137.16)
-		(end 101.6 148.59)
+		(start 74.93 138.43)
+		(end 104.14 149.86)
 		(stroke
 			(width 0)
@@
 	(text "Wires to \"snap\" connectors on M48T59Y-70MH1"
 		(exclude_from_sim no)
-		(at 49.022 151.638 0)
+		(at 66.294 153.416 0)
 		(effects
 			(font
@@
 			)
 			(justify left)
-		)
-	)
-	(symbol
-		(lib_id "Device:Crystal")
-		(at 50.8 130.81 0)
-		(unit 1)
-		(exclude_from_sim no)
-		(in_bom yes)
-		(on_board yes)
-		(dnp no)
-		(fields_autoplaced yes)
-		(property "Reference" "Y1"
-			(at 50.8 123.19 0)
-			(effects
-				(font
-					(size 1.27 1.27)
-				)
-			)
-		)
-		(property "Value" "32.768 kHz"
-			(at 50.8 125.73 0)
-			(effects
-				(font
-					(size 1.27 1.27)
-				)
-			)
-		)
-		(property "Footprint" "Crystal:Crystal_C38-LF_D3.0mm_L8.0mm_Horizontal"
-			(at 50.8 130.81 0)
-			(effects
-				(font
-					(size 1.27 1.27)
-				)
-				(hide yes)
-			)
-		)
-		(property "Datasheet" "~"
-			(at 50.8 130.81 0)
-			(effects
-				(font
-					(size 1.27 1.27)
-				)
-				(hide yes)
-			)
-		)
-		(property "Description" "Two pin crystal"
-			(at 50.8 130.81 0)
-			(effects
-				(font
-					(size 1.27 1.27)
-				)
-				(hide yes)
-			)
-		)
-		(pin "2"
-		)
-		(pin "1"
-		)
-		(instances
-			(project ""
-				(path "/a5619b9c-2a1e-4dd3-8c34-92032ec8ab73"
-					(reference "Y1")
-					(unit 1)
-				)
-			)
 		)
 	)
@@
 					(unit 1)
 				)
-			)
-		)
-	)
-	(symbol
-		(lib_id "Connector:Conn_01x02_Pin")
-		(at 49.53 144.78 90)
-		(unit 1)
-		(exclude_from_sim no)
-		(in_bom yes)
-		(on_board yes)
-		(dnp no)
-		(fields_autoplaced yes)
-		(property "Reference" "J3"
-			(at 53.34 142.8749 90)
-			(effects
-				(font
-					(size 1.27 1.27)
-				)
-				(justify right)
-			)
-		)
-		(property "Value" "Conn_01x02_Pin"
-			(at 53.34 145.4149 90)
-			(effects
-				(font
-					(size 1.27 1.27)
-				)
-				(justify right)
-			)
-		)
-		(property "Footprint" "Connector_PinHeader_2.54mm:PinHeader_1x02_P2.54mm_Vertical"
-			(at 49.53 144.78 0)
-			(effects
-				(font
-					(size 1.27 1.27)
-				)
-				(hide yes)
-			)
-		)
-		(property "Datasheet" "~"
-			(at 49.53 144.78 0)
-			(effects
-				(font
-					(size 1.27 1.27)
-				)
-				(hide yes)
-			)
-		)
-		(property "Description" "Generic connector, single row, 01x02, script generated"
-			(at 49.53 144.78 0)
-			(effects
-				(font
-					(size 1.27 1.27)
-				)
-				(hide yes)
-			)
-		)
-		(pin "1"
-		)
-		(pin "2"
-		)
-		(instances
-			(project ""
-				(path "/a5619b9c-2a1e-4dd3-8c34-92032ec8ab73"
-					(reference "J3")
-					(unit 1)
-				)
